Commit message: add rqt, controller

File: mybot_description/urdf/macros.xacro (robot description, xacro)
@@ -21,50 +21,51 @@
 	</macro>
 	<macro name="wheel" params="lr tY">
-	<link name="${lr}_wheel">
-	  <collision>
-	    <origin xyz="0 0 0" rpy="0 ${PI/2} ${PI/2}" />
-	    <geometry>
-	      <cylinder length="${wheelWidth}" radius="${wheelRadius}"/>
-	    </geometry>
-	  </collision>
-	  <visual>
-	    <origin xyz="0 0 0" rpy="0 ${PI/2} ${PI/2}" />
-	    <geometry>
-	      <cylinder length="${wheelWidth}" radius="${wheelRadius}"/>
-	    </geometry>
-	    <material name="black"/>
-	  </visual>
-	  <inertial>
-	    <origin xyz="0 0 0" rpy="0 ${PI/2} ${PI/2}" />
-	    <mass value="${wheelMass}"/>
-	    <cylinder_inertia m="${wheelMass}" r="${wheelRadius}" h="${wheelWidth}"/>
-	  </inertial>
-	</link>
-	<gazebo reference="${lr}_wheel">
-	  <mu1 value="1.0"/>
-	  <mu2 value="1.0"/>
-	  <kp  value="10000000.0" />
-	  <kd  value="1.0" />
-	  <fdir1 value="1 0 0"/>
-	  <material>Gazebo/Black</material>
-	</gazebo>
-	<joint name="${lr}_wheel_hinge" type="continuous">
-	  <parent link="chassis"/>
-	  <child link="${lr}_wheel"/>
-	<origin xyz="${-wheelPos+chassisLength/2} ${tY*wheelWidth/2+tY*chassisWidth/2} ${wheelRadius}" rpy="0 0 0" />
-	  <axis xyz="0 1 0" rpy="0 0 0" />
-	  <limit effort="100" velocity="100"/>
-	  <joint_properties damping="0.0" friction="0.0"/>
-	</joint>
-	<transmission name="${lr}_trans">
-	  <type>transmission_interface/SimpleTransmission</type>
-	  <joint name="${lr}_wheel_hinge">
-	      <hardwareInterface>EffortJointInterface</hardwareInterface>
-	  </joint>
-	  <actuator name="${lr}Motor">
-	    <hardwareInterface>EffortJointInterface</hardwareInterface>
-	    <mechanicalReduction>10</mechanicalReduction>
-	  </actuator>
-	</transmission>
+		<link name="${lr}_wheel">
+		  <collision>
+		    <origin xyz="0 0 0" rpy="0 ${PI/2} ${PI/2}" />
+		    <geometry>
+		      <cylinder length="${wheelWidth}" radius="${wheelRadius}"/>
+		    </geometry>
+		  </collision>
+		  <visual>
+		    <origin xyz="0 0 0" rpy="0 ${PI/2} ${PI/2}" />
+		    <geometry>
+		      <cylinder length="${wheelWidth}" radius="${wheelRadius}"/>
+		    </geometry>
+		    <material name="black"/>
+		  </visual>
+		  <inertial>
+		    <origin xyz="0 0 0" rpy="0 ${PI/2} ${PI/2}" />
+		    <mass value="${wheelMass}"/>
+		    <cylinder_inertia m="${wheelMass}" r="${wheelRadius}" h="${wheelWidth}"/>
+		  </inertial>
+		</link>
+		<gazebo reference="${lr}_wheel">
+		  <mu1 value="1.0"/>
+		  <mu2 value="1.0"/>
+		  <kp  value="10000000.0" />
+		  <kd  value="1.0" />
+		  <fdir1 value="1 0 0"/>
+		  <material>Gazebo/Black</material>
+		</gazebo>
+		<joint name="${lr}_wheel_hinge" type="continuous">
+		  <parent link="chassis"/>
+		  <child link="${lr}_wheel"/>
+		  <origin xyz="${-wheelPos+chassisLength/2} ${tY*wheelWidth/2+tY*chassisWidth/2} ${wheelRadius}" rpy="0 0 0" />
+		  <axis xyz="0 1 0" rpy="0 0 0" />
+		  <limit effort="100000" velocity="100000"/>
+		  <joint_properties damping="0.0" friction="0.0"/>
+		</joint>
+<!--The <transmission> element is used to link actuators to joints -->
+		<transmission name="${lr}_trans">
+		  <type>transmission_interface/SimpleTransmission</type>
+		  <joint name="${lr}_wheel_hinge">
+		      <hardwareInterface>EffortJointInterface</hardwareInterface>
+		  </joint>
+		  <actuator name="${lr}Motor">
+		    <hardwareInterface>EffortJointInterface</hardwareInterface>
+		    <mechanicalReduction>10</mechanicalReduction>
+		  </actuator>
+		</transmission>
 	</macro>
 </robot>

File: mybot_description/urdf/mybot.xacro (robot description, xacro)
@@ -70,3 +70,27 @@
 	<wheel lr="left" tY="1"/>
 	<wheel lr="right" tY="-1"/>
+	<joint name="cam_joint" type="fixed">
+	  <parent link="chassis"/>
+	  <child link="camera"/>
+	</joint>
+	<link name="camera">
+	  <collision>
+	    <origin xyz="0 0 0.2" rpy="0 0 0"/>
+	    <geometry>
+	      <box size="${cameraSize} ${cameraSize} ${cameraSize}"/>
+	    </geometry>
+	  </collision>
+	  <visual>
+	    <origin xyz="0 0 0.2" rpy="0 0 0"/>
+	    <geometry>
+	      <box size="${cameraSize} ${cameraSize} ${cameraSize}"/>
+	    </geometry>
+	    <material name="blue"/>
+	  </visual>
+	  <inertial>
+	    <mass value="${cameraMass}" />
+	    <origin xyz="0 0 0.2" rpy="0 0 0"/>
+	    <box_inertia m="${cameraMass}" x="${cameraSize}" y="${cameraSize}" z="${cameraSize}" />
+	  </inertial>
+	</link>
 </robot>
